File: electrical/boards/voltage-current-sensor/Voltage_current_monitor_schematic.kicad_pcb (KiCad board)
At the start: 2 copper layers, 49.5 x 43.5 mm, 13 parts, among them IC1 INA236AIDDFR, J1 Conn_01x06_Female, J2 691137710006 terminal block

Commit message: Add Aerial KiCad library and fix voltage-current board
Parts:
- IC1: footprint Symbol:SOP65P280X110-8N -> RSX_Aerial:SOP65P280X110-8N
- J1: footprint rsx_headers:PinSocket_1x06_P2.54mm_Vertical -> RSX_Aerial:PinSocket_1x06_P2.54mm_Vertical
- J2: footprint Connector:691137710006 -> RSX_Aerial:691137710006
- R1, R2, R3: footprint rsx_resistors:R_0603_1608Metric -> RSX_Aerial:R_0603_1608Metric
- R4: footprint rsx_resistors:R_1206_3216Metric -> RSX_Aerial:R_1206_3216Metric
Connections:
- IC1 pad 3: Net-(IC1-GND) -> GND
- TP5 pad 1: Net-(IC1-GND) -> GND
Routing:
- net Net-(IC1-GND): track 23.2 -> 0.00 mm, vias 2 -> 0
- net GND: track 48.7 -> 72.0 mm, vias 2 -> 4
