File: electrical/boards/voltage-current-sensor/Voltage_current_monitor_schematic.kicad_sch (KiCad schematic)
At the start: 6 parts, among them IC1 INA236AIDDFR

Commit message: Add Aerial KiCad library and fix voltage-current board
Parts:
- added J1: Conn_01x06_Female, RSX_Aerial:PinSocket_1x06_P2.54mm_Vertical, symbol RSX_Aerial_Headers:Conn_01x06_Female
- added J2: 691137710006 terminal block, RSX_Aerial:691137710006, symbol Connector_Generic:Conn_01x06
- added TP1: IN+, TestPoint:TestPoint_Loop_D2.50mm_Drill1.0mm, symbol Connector:TestPoint
- added TP2: IN-, TestPoint:TestPoint_Loop_D2.50mm_Drill1.0mm, symbol Connector:TestPoint
- added TP3: SDA, TestPoint:TestPoint_Loop_D2.50mm_Drill1.0mm, symbol Connector:TestPoint
- added TP4: SCL, TestPoint:TestPoint_Loop_D2.50mm_Drill1.0mm, symbol Connector:TestPoint
- added TP5: GND, TestPoint:TestPoint_Loop_D2.50mm_Drill1.0mm, symbol Connector:TestPoint
- C2: symbol rsx_Capacitors:0u1_0402 -> RSX_Aerial_Capacitors:0u1_0402
- IC1: footprint SOP65P280X110-8N -> RSX_Aerial:SOP65P280X110-8N; symbol Power_Management:INA236AIDDFR -> RSX_Aerial:INA236AIDDFR
- R1, R2, R3: footprint rsx_resistors:R_0603_1608Metric -> RSX_Aerial:R_0603_1608Metric; symbol rsx_Resistors:4K7 -> RSX_Aerial_Resistors:4K7
- R4: footprint rsx_resistors:R_1206_3216Metric -> RSX_Aerial:R_1206_3216Metric; symbol rsx_Resistors:0R100 1/2W -> RSX_Aerial_Resistors:0R100 1/2W
Connections:
- net 3.3V: now also J1.1 (Pin_1)
- net Bus voltage: now also J2.5 (Pin_5), J2.6 (Pin_6), TP1.1
- net GND: now also J1.2 (Pin_2), J1.6 (Pin_6), J2.1 (Pin_1), J2.2 (Pin_2), TP5.1
- net Load: now also J2.3 (Pin_3), J2.4 (Pin_4), TP2.1
- net SCL: now reaches IC1.5 (SCL), R2.1
- net SCL: now also J1.4 (Pin_4), TP4.1
- net SDA: now reaches IC1.6 (SDA), R1.1
- net SDA: now also J1.3 (Pin_3), TP3.1
- net Alert: now reaches IC1.8 (ALERT), R3.1
- net Alert: now also J1.5 (Pin_5)
Other:
- note added: "Bus / load terminal"
- note added: "I2C header"
- note added: "Test points"
