File: electrical/blocks/Voltage_current_monitor_schematic.kicad_sch (KiCad schematic)
At the start: 6 parts, among them IC1 INA236AIDDFR

Commit message: Relink blocks to Aerial library
Parts:
- C2: footprint Capacitor_SMD:C_01005_0402Metric -> RSX_Aerial:C_0603_1608Metric; symbol rsx_Capacitors:0u1_0402 -> RSX_Aerial_Capacitors:0u1; DPN 1276-1043-1-ND -> 445-1314-1-ND; MFR Samsung Electro-Mechanics -> TDK Corporation; MPN CL05A104KA5NNNC -> C1608X7R1H104K080AA
- IC1: footprint SOP65P280X110-8N -> RSX_Aerial:SOP65P280X110-8N; symbol Power_Management:INA236AIDDFR -> RSX_Aerial:INA236AIDDFR
- R1, R2, R3: footprint rsx_resistors:R_0603_1608Metric -> RSX_Aerial:R_0603_1608Metric; symbol rsx_Resistors:4K7 -> RSX_Aerial_Resistors:4K7
- R4: footprint rsx_resistors:R_1206_3216Metric -> RSX_Aerial:R_1206_3216Metric; symbol rsx_Resistors:0R100 1/2W -> RSX_Aerial_Resistors:0R100 1/2W
